Commit message: change joint type joint4

File: Examples/test.urdf (robot description, URDF)
Before this commit: robot test, 4 links, 3 joints
Joints:
- joint second_to_third_joint: limit (none) -> lower=-2 upper=2 effort=500 velocity=10
- joint third_to_forth_joint: origin xyz=0 0 0.5 rpy=0 0 0 -> xyz=-0.5 0 0.5 rpy=0 0 0
